File: tarea 3/NIZAO/BoardNIZAO.kicad_sch (KiCad schematic)
At the start: 1 part, among them U1 ESP32-S3-WROOM-1

Commit message: Actualizan y creando tarea 4
Parts:
- added C1: 100nf, Capacitor_SMD:C_0603_1608Metric, symbol Capacitor_AKL:C_0603
- added C2, C3: 100NF, Capacitor_SMD:C_0603_1608Metric, symbol Capacitor_AKL:C_0603
- added J5: PZ254R-12-14P, XFCN PZ254R-12-14P:HDR-TH_14P-P2.54-H-M-R2-C7-S2.54, symbol EasyEDA:PZ254R-12-14P
- added LED1: LED_0603_Red, LED_SMD:LED_0603_1608Metric, symbol LED_AKL:LED_0603_Red
- added R1, R2: R_0603, Resistor_SMD:R_0603_1608Metric, symbol Resistor_US_AKL:R_0603
- added R3: 22K, Resistor_SMD:R_0603_1608Metric, symbol Resistor_US_AKL:R_0603
- added R4: 2.2K, Resistor_SMD:R_0603_1608Metric, symbol Resistor_US_AKL:R_0603
- added SW1: TS-1088-AR02016, XUNPU TS-1088-AR02016:SW-SMD_L3.9-W3.0-P4.45, symbol EasyEDA:TS-1088-AR02016
- added TP1, TP2, TP3, TP4: TestPoint, TestPoint:TestPoint_THTPad_D1.5mm_Drill0.7mm, symbol Connector:TestPoint
- added U1: ADS1115IDGS, Package_SO:TSSOP-10_3x3mm_P0.5mm, symbol Analog_ADC:ADS1115IDGS
- added U3: RS485-PROTECT, RS485-PROTECT:RS-485-PROTECT, symbol MG_CONNECTORS:RS485-PROTECT
- U2: renamed from U1; footprint RF_Module:ESP32-S3-WROOM-1 -> RF_Module:ESP32-S3-WROOM-1U
Connections:
- net GND: now reaches U2.1 (GND), U2.40 (GND), U2.41 (GND)
- net GND: now also C1.2, C2.1, C3.2, J5.13, J5.14, LED1.1 (K), R2.2, SW1.2, U1.1 (ADDR), U1.3 (GND), U3.2 (GND)
- net i2c_sda: now reaches U2.10 (IO17)
- net i2c_sda: now also J5.8, U1.9 (SDA)
- net i2c_scl: now reaches U2.11 (IO18)
- net i2c_scl: now also J5.10, U1.10 (SCL)
- net rs485_rx: now reaches U2.12 (IO8)
- net usb-: now reaches U2.13 (USB_D-)
- net usb-: now also J5.6
- net usb+: now reaches U2.14 (USB_D+)
- net usb+: now also J5.4
- net IN_NPN4: now reaches U2.15 (IO3)
- net OUT_PNP1: now reaches U2.16 (IO46)
- net rs485_tx: now reaches U2.17 (IO9)
- net rs485-com: now reaches U2.18 (IO10)
- net cs: now reaches U2.19 (IO11)
- net cs: now also J5.3
- net +3.3V: now reaches U2.2 (3V3)
- net +3.3V: now also C3.1, J5.2, R3.2, U1.8 (VDD), U3.1 (VCC)
- net miso: now reaches U2.20 (IO12)
- net miso: now also J5.7
- net mosi: now reaches U2.21 (IO13)
- net mosi: now also J5.5
- net clk: now reaches U2.22 (IO14)
- net clk: now also J5.9
- net LED_INFO: now reaches U2.23 (IO21)
- net LED_INFO: now also R4.2
- net OUT_PNP2: now reaches U2.24 (IO47)
- net TEMP_CS: now reaches U2.25 (IO48)
- net OUT_RLY2: now reaches U2.26 (IO45)
- net IN_NPN1: now reaches U2.27 (IO0)
- net EN: now reaches U2.3 (EN)
- net EN: now also C2.2, R3.1, SW1.1
- net OUT_NPN1: now reaches U2.31 (IO38)
- net OUT_NPN2: now reaches U2.32 (IO39)
- net OUT_NPN3: now reaches U2.33 (IO40)
- net OUT_NPN4: now reaches U2.34 (IO41)
- net OUT_RLY1: now reaches U2.35 (IO42)
- net EMRX: now reaches U2.36 (RXD0)
- net EM_TX: now reaches U2.37 (TXD0)
- net IN_NPN3: now reaches U2.38 (IO2)
- net IN_NPN2: now reaches U2.39 (IO1)
- net IN_PNP1: now reaches U2.4 (IO4)
- net IN_PNP2: now reaches U2.5 (IO5)
- net IN_VDC_ADC: now reaches U2.6 (IO6)
- net IN_VDC_ADC: now also C1.1, R1.2, R2.1
- net acc_cs: now reaches U2.7 (IO7)
- net GPIO1: now reaches U2.8 (IO15)
- net GPIO1: now also J5.11
- net GPIO2: now reaches U2.9 (IO16)
- net GPIO2: now also J5.12
- new net: LED1.2 (A), R4.1
- new net +24V: R1.1
- new net +5V: J5.1
- new net CON_RS485_A: U3.7 (A)
- new net CON_RS485_B: U3.8 (B)
- new net CON_RS485_G: U3.6 (RGND)
- new net IN-0-10V/OUT3V: TP3.1, U1.6 (AIN2)
- new net IN-0-10V1/OUT3V: TP4.1, U1.7 (AIN3)
- new net IN-4-20MA/OUT: TP1.1, U1.4 (AIN0)
- new net IN-4-20MA1/OUT: TP2.1, U1.5 (AIN1)
- new net RS485-CON: U3.5 (CON)
- new net RS485-RX: U3.4 (RXD)
- new net RS485-TX: U3.3 (TXD)
- no-connect marks 0 -> 3
Other:
- added sheet EnergyMeterA1 (EnergyMeterA1.kicad_sch)
- added sheet IN-0-10V (IN-0-10V.kicad_sch)
- added sheet IN-0-10V1 (IN-0-10V.kicad_sch)
- added sheet IN-4-20MA (IN-4-20MA.kicad_sch)
- added sheet IN-4-20MA1 (IN-4-20MA.kicad_sch)
- added sheet IN-DI (IN-DI.kicad_sch)
- added sheet IN-DI1 (IN-DI.kicad_sch)
- added sheet IN-DI2 (IN-DI.kicad_sch)
- added sheet IN-DI3 (IN-DI.kicad_sch)
- added sheet IN-DI4 (IN-DI.kicad_sch)
- added sheet IN-DI5 (IN-DI.kicad_sch)
- added sheet OUT-0-10V (OUT-0-10V.kicad_sch)
- added sheet OUT-4-20MA (OUT-4-20MA.kicad_sch)
- added sheet OUT-NPN (OUT-NPN.kicad_sch)
- added sheet OUT-NPN1 (OUT-NPN.kicad_sch)
- added sheet OUT-NPN2 (OUT-NPN.kicad_sch)
- added sheet OUT-NPN3 (OUT-NPN.kicad_sch)
- added sheet OUT-PNP (OUT-PNP.kicad_sch)
- added sheet RLY (RLY.kicad_sch)
- added sheet TC (TC.kicad_sch)
- moved on the sheet: U2
