File: tarea 3/NIZAO/NIZAO.kicad_sch (KiCad schematic)
At the start: 0 parts

Commit message: Actualizo tarea 3
Parts:
- added J1, J2, J3, J4: Screw_Terminal_01x09, symbol Connector:Screw_Terminal_01x09
Connections:
- new net CON_IN-0-10V_1: J2.2 (Pin_2)
- new net CON_IN-0-10V_2: J2.3 (Pin_3)
- new net CON_IN-4-20MA_1: J2.4 (Pin_4)
- new net CON_IN-4-20MA_2: J2.5 (Pin_5)
- new net CON_IN_CT_P: J2.9 (Pin_9)
- new net CON_IN_NPN1: J1.3 (Pin_3)
- new net CON_IN_NPN2: J1.4 (Pin_4)
- new net CON_IN_NPN3: J1.5 (Pin_5)
- new net CON_IN_NPN4: J1.6 (Pin_6)
- new net CON_IN_PNP1: J1.7 (Pin_7)
- new net CON_IN_PNP2: J1.8 (Pin_8)
- new net CON_IN_TC+: J1.9 (Pin_9)
- new net CON_IN_TC-: J2.1 (Pin_1)
- new net CON_IN_VAC_N: J2.6 (Pin_6)
- new net CON_IN_VAC_P: J2.7 (Pin_7)
- new net CON_OUT_0-10V: J4.8 (Pin_8)
- new net CON_OUT_4-20MA: J4.7 (Pin_7)
- new net CON_OUT_NPN_1: J3.6 (Pin_6)
- new net CON_OUT_NPN_2: J3.7 (Pin_7)
- new net CON_OUT_NPN_3: J3.8 (Pin_8)
- new net CON_OUT_NPN_4: J3.9 (Pin_9)
- new net CON_OUT_PNP_1: J3.4 (Pin_4)
- new net CON_OUT_PNP_2: J3.5 (Pin_5)
- new net CON_OUT_RLY1_COM: J4.1 (Pin_1)
- new net CON_OUT_RLY1_NC: J4.2 (Pin_2)
- new net CON_OUT_RLY1_NO: J4.3 (Pin_3)
- new net CON_OUT_RLY2_COM: J4.4 (Pin_4)
- new net CON_OUT_RLY2_NC: J4.5 (Pin_5)
- new net CON_OUT_RLY2_NO: J4.6 (Pin_6)
- new net CON_RS485_A: J3.2 (Pin_2)
- new net CON_RS485_B: J3.3 (Pin_3)
- new net CON_RS485_G: J3.1 (Pin_1)
- new net CO_IN_CT_N: J2.8 (Pin_8)
- new net GND: J1.2 (Pin_2), J4.9 (Pin_9)
- new net VCC_IN: J1.1 (Pin_1)
Other:
- added sheet BoardNIZAO (BoardNIZAO.kicad_sch)
- added sheet PawerSupply (PawerSupply.kicad_sch)

Commit message: Actualizan y creando tarea 4
Parts:
- added H1, H2: MountingHole, MountingHole:MountingHole_3.2mm_M3, symbol Mechanical:MountingHole
- J1, J2, J3, J4: footprint (none) -> TerminalBlock_Phoenix:TerminalBlock_Phoenix_PT-1,5-9-5.0-H_1x09_P5.00mm_Horizontal
Connections:
- net CON_IN-0-10V_1 renamed BoardNIZAO/CON_IN_0-10V_1
- net CON_IN-0-10V_2 renamed BoardNIZAO/CON_IN_0-10V_2
- net CON_IN-4-20MA_1 renamed BoardNIZAO/CON-IN-4-20MA_1
- net CON_IN-4-20MA_2 renamed BoardNIZAO/CON-IN-4-20MA_2
- net CON_IN_CT_P renamed BoardNIZAO/CON-IN_VAC_P
- net CON_IN_NPN1 renamed BoardNIZAO/CON_IN_NPN1
- net CON_IN_NPN2 renamed BoardNIZAO/CON_IN_NPN2
- net CON_IN_NPN3 renamed BoardNIZAO/CON_IN_NPN3
- net CON_IN_NPN4 renamed BoardNIZAO/CON_IN_NPN4
- net CON_IN_PNP1 renamed BoardNIZAO/CON_IN_PNP1
- net CON_IN_PNP2 renamed BoardNIZAO/CON_IN_PNP2
- net CON_IN_TC+ renamed BoardNIZAO/CON_IN_TC+
- net CON_IN_TC- renamed BoardNIZAO/CON_IN_TC-
- net CON_IN_VAC_N renamed BoardNIZAO/CON-IN_CT_N
- net CON_IN_VAC_P renamed BoardNIZAO/CON-IN_CT_P
- net CON_OUT_0-10V renamed BoardNIZAO/CON_OUT_0-10V
- net CON_OUT_4-20MA renamed BoardNIZAO/CON_OUT_4-20MA
- net CON_OUT_NPN_1 renamed BoardNIZAO/CON_OUT_NPN_3
- net CON_OUT_NPN_2 renamed BoardNIZAO/CON_OUT_NPN_4
- net CON_OUT_NPN_3 renamed BoardNIZAO/CON_OUT_PNP_1
- net CON_OUT_NPN_4 renamed BoardNIZAO/CON_OUT_PNP_2
- net CON_OUT_PNP_1 renamed BoardNIZAO/CON_OUT_NPN_1
- net CON_OUT_PNP_2 renamed BoardNIZAO/CON_OUT_NPN_2
- net CON_OUT_RLY1_COM renamed BoardNIZAO/CON_OUT_RLY1_COM
- net CON_OUT_RLY1_NC renamed BoardNIZAO/CON_OUT_RLY1_NC
- net CON_OUT_RLY1_NO renamed BoardNIZAO/CON_OUT_RLY1_NO
- net CON_OUT_RLY2_COM renamed BoardNIZAO/CON_OUT_RLY2_NC
- net CON_OUT_RLY2_NC renamed BoardNIZAO/CON_OUT_RLY2_NO
- net CON_OUT_RLY2_NO renamed BoardNIZAO/CON_OUT_RLY2_COM
- net CON_RS485_A renamed BoardNIZAO/CON_RS485_A
- net CON_RS485_B renamed BoardNIZAO/CON_RS485_B
- net CON_RS485_G renamed BoardNIZAO/CON_RS485_G
- net CO_IN_CT_N renamed Earth
- net VCC_IN renamed +24V
Other:
- sheet BoardNIZAO ports: added CON-IN-4-20MA_1, CON-IN-4-20MA_2, CON-IN_CT_N, CON-IN_CT_P, CON-IN_VAC_N, CON-IN_VAC_P, CON_IN_0-10V_1, CON_IN_0-10V_2, CON_IN_NPN1, CON_IN_NPN2, CON_IN_NPN3, CON_IN_NPN4, CON_IN_PNP1, CON_IN_PNP2, CON_IN_TC+, CON_IN_TC-, CON_OUT_0-10V, CON_OUT_4-20MA, CON_OUT_NPN_1, CON_OUT_NPN_2, CON_OUT_NPN_3, CON_OUT_NPN_4, CON_OUT_PNP_1, CON_OUT_PNP_2, CON_OUT_RLY1_COM, CON_OUT_RLY1_NC, CON_OUT_RLY1_NO, CON_OUT_RLY2_COM, CON_OUT_RLY2_NC, CON_OUT_RLY2_NO, CON_RS485_A, CON_RS485_B, CON_RS485_G; removed none
- sheet PawerSupply ports: added VCC_IN; removed none
- moved on the sheet: J1, J2, J3, J4
