File: tarea 3/NIZAO/PawerSupply.kicad_sch (KiCad schematic)
At the start: 0 parts

Commit message: Actualizan y creando tarea 4
Parts:
- added C10, C9: 22uF, Capacitor_SMD:C_0805_2012Metric, symbol Capacitor_AKL:C_0805
- added C11, C12, C6: 47UF, Capacitor_SMD:CP_Elec_6.3x7.7, symbol MG_CAPACITOR:CAP-POL-SMD-47UF-16V-D6.3MM
- added C7: 10uF, Capacitor_SMD:C_0805_2012Metric, symbol Capacitor_AKL:C_0805
- added C8: 100NF, Capacitor_SMD:C_0805_2012Metric, symbol Capacitor_AKL:C_0805
- added D3, D4: SS14, Diode_SMD:D_SMA, symbol Diode:SS14
- added D5: SMF24CA, Diode_SMD:D_SOD-123F, symbol Diode_TVS_AKL:SMF24CA
- added D6: SMF3.3, SMF3.3_SODFL3718X108N:SMF3.3_SODFL3718X108N, symbol Snapeda:SMF3.3
- added L1: 10uH, Inductor_SMD:L_APV_APH0630, symbol Device:L_Ferrite
- added TP5, TP6, TP7: TestPoint_Hole1, TestPoint:TestPoint_THTPad_D1.5mm_Drill0.7mm, symbol MG_ELECTROMECANICAL:TestPoint_Hole1
- added U4: AP63203WU, Package_TO_SOT_SMD:TSOT-23-6, symbol Regulator_Switching:AP63203WU
Connections:
- new net: C8.1, U4.6 (BST)
- new net +3.3V: C10.1, C11.1, C12.1, C9.1, D6.A, L1.2, U4.1 (FB)
- new net +5V: D3.2 (A), TP6.1
- new net GND: C10.2, C11.2, C12.2, C6.2, C7.2, C9.2, D5.1 (K), D6.C, U4.4 (GND)
- new net VCC_IN: C6.1, D4.2 (A), TP5.1
- new net sw: C8.2, L1.1, U4.5 (SW)
- new net vdc_in: C7.1, D3.1 (K), D4.1 (K), D5.2 (A), TP7.1, U4.2 (EN), U4.3 (IN)
Other:
- note added: "usar X5R"
