File: tarea 4/NIZAO_Board_Vertical/NIZAO_Board_Vertical.kicad_sch (KiCad schematic)
At the start: 1 part

Commit message: actualizacion
Parts:
- removed H1: PZ254R-12-14P, easyeda2kicad:HDR-TH_14P-P2.54-H-M-R2-C7-S2.54, symbol easyeda2kicad:PZ254R-12-14P
- added C1: 47uF, Capacitor_SMD:C_0603_1608Metric, symbol Capacitor_AKL:C_0603
- added C2: 100nF, Capacitor_SMD:C_0603_1608Metric, symbol Capacitor_AKL:C_0603
- added Card1: TF-115, EasyEDA:TF-SMD_TF-115, symbol EasyEDA:TF-115
- added FPC1: FPC-05FB-30PH20, EasyEDA:FPC-SMD_30P-P0.50_FPC-05FB-30PH20, symbol EasyEDA:FPC-05FB-30PH20
- added J1: PZ254R-12-14P, EasyEDA:HDR-TH_14P-P2.54-H-M-R2-C7-S2.54, symbol EasyEDA:PZ254R-12-14P
- added L1: 600 Ohm, Capacitor_SMD:C_0805_2012Metric, symbol SparkFun-Coil:Ferrite_600Ohm_0805_500mA
- added R1, R2: 5.1k, Resistor_SMD:R_0603_1608Metric, symbol Resistor_US_AKL:R_0603
- added R3, R9: 10K, Resistor_SMD:R_0603_1608Metric, symbol Resistor_US_AKL:R_0603
- added R4, R5, R8: 2.2K, Resistor_SMD:R_0603_1608Metric, symbol Resistor_US_AKL:R_0603
- added R6: 10R, Resistor_SMD:R_0603_1608Metric, symbol Resistor_US_AKL:R_0603
- added R7: 220R, Resistor_SMD:R_0603_1608Metric, symbol Resistor_US_AKL:R_0603
- added U1: MC-121-L119, EasyEDA:USB-C-SMD_HANBO_MC-121-L119, symbol EasyEDA:MC-121-L119
Connections:
- new net: R1.1, U1.A5 (CC1)
- new net: C1.1, C2.1, Card1.4 (VDD), L1.1
- new net: R2.1, U1.B5 (CC2)
- new net: Card1.7 (DAT0), R7.2
- new net: Card1.5 (CLK), R6.2
- new net: Card1.1 (DAT2), R8.2
- new net: Card1.2 (CD/DAT3), R9.2
- new net: Card1.8 (DAT1), R4.2
- new net +3.3V: J1.2, L1.2, R3.1, R4.1, R5.1, R8.1, R9.1
- new net +5V: J1.1, U1.A4B9 (VBUS), U1.B4A9 (VBUS)
- new net GND: C1.2, C2.2, Card1.10 (SHELL), Card1.11 (SHELL), Card1.12 (SHELL), Card1.13 (SHELL), Card1.6 (VSS), J1.13, J1.14, R1.2, R2.2, U1.13 (EH), U1.A1B12 (GND), U1.B1A12 (GND)
- new net GPIO1: J1.11
- new net GPIO2: J1.12
- new net clk: J1.9, R6.1
- new net cs: J1.3
- new net i2c_scl: J1.10
- new net i2c_sda: J1.8
- new net miso: J1.7, R5.2, R7.1
- new net mosi: Card1.3 (CMD), J1.5, R3.2
- new net usb+: J1.4, U1.A6 (DP1), U1.B6 (DP2)
- new net usb-: J1.6, U1.A7 (DN1), U1.B7 (DN2)
- no-connect marks 0 -> 3
Other:
- removed sheet NIZAO_Board_Vertical
