File: NIZAO/IN-0-10V.kicad_sch (KiCad schematic)
At the start: 5 parts

Commit message: Colocandos los 3d de los componetes en la placa NIZAO
Parts:
- D7: footprint DIODES BAT54S-7-F:SOT-23_L2.9-W1.3-P1.90-LS2.4-BR -> JLCImport:BAT54S-7-F
