File: NIZAO/IN-4-20MA.kicad_sch (KiCad schematic)
At the start: 8 parts

Commit message: Colocandos los 3d de los componetes en la placa NIZAO
Parts:
- D1: footprint DIODES 1N5819HW-7-F:SOD-123_L2.7-W1.6-LS3.7-RD -> JLCImport:1N5819HW-7-F; symbol EasyEDA:1N5819HW-7-F -> JLCImport:1N5819HW-7-F; LCSC (none) -> C82544; Manufacturer (none) -> Diodes Incorporated; Manufacturer Part (none) -> 1N5819HW-7-F
