File: NIZAO/TC.kicad_sch (KiCad schematic)
At the start: 15 parts, among them U11 MAX31856MUD+

Commit message: Colocandos los 3d de los componetes en la placa NIZAO
Parts:
- U11: footprint MAXIM MAX31856MUD+:TSSOP-14_L5.0-W4.4-P0.65-LS6.4-BL -> JLCImport:MAX31856MUD
